File: hardware/master-pcb-easyeda/kicad/ESP32-S3-Master-PCB.kicad_sch (KiCad schematic)
At the start: 70 parts, among them J1 Screw Terminal 2P, J10 ARM Debug 2x5, J11 Header 1x6 RA, J12 JST-PH 2P, J13 JST-PH 2P, J14 JST-XH 5P, J15 JST-XH 5P, J16 JST-XH 5P, J17 JST-XH 5P, J18 JST-XH 5P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

Commit message: v1.3.0: Add water temperature sensor support with display widget
Parts:
- added C17: 100nF, symbol 100nF_C17
- added C18: 100nF, symbol 100nF_C18
- added D5: BZT52C3V3, symbol BZT52C3V3_D5
- added J19: JST-PH 2P, symbol JST-PH_2P_J19
- added R27: 1K, symbol 1K_R27
- added R28: 10K, symbol 10K_R28
- added R29: 1K, symbol 1K_R29
